File: NovaPlay3_KiCad/Memory.kicad_sch (KiCad schematic)
At the start: 0 parts

Commit message: Finished power management
power management schematic is done
Parts:
- added U2: M95P32-IXMNT/E, symbol CPU_NXP_IMX:M95P32-IXMNT/E
Connections:
- new net +3.3V: U2.3 (~{W}-DQ2), U2.7 (~{HOLD}-DQ3), U2.8 (VCC)
- new net EEPROM_CS: U2.1 (~{S})
- new net GND: U2.4 (GND)
- new net MISO: U2.2 (Q-DQ1)
- new net MOSI: U2.5 (D-DQ0)
- new net SCK: U2.6 (C)

Commit message: Sync
Parts:
- renumbered U2 to U4
Changed lines of the file:
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@@
 		(dnp no)
 		(fields_autoplaced yes)
-		(property "Reference" "U2"
+		(property "Reference" "U4"
 			(at 121.5233 86.36 0)
 			(effects
@@
 			(project "NovaPlay3"
 				(path "/3902e32d-76e7-44cb-8277-c0e17db8d088/d1d82891-0be9-49d5-808b-34296a85b88c"
-					(reference "U2")
+					(reference "U4")
 					(unit 1)
 				)
@@
 		(dnp no)
 		(fields_autoplaced yes)
-		(property "Reference" "#PWR07"
+		(property "Reference" "#PWR026"
 			(at 86.36 101.6 0)
 			(effects
@@
 			(project "NovaPlay3"
 				(path "/3902e32d-76e7-44cb-8277-c0e17db8d088/d1d82891-0be9-49d5-808b-34296a85b88c"
-					(reference "#PWR07")
+					(reference "#PWR026")
 					(unit 1)
 				)
@@
 		(dnp no)
 		(fields_autoplaced yes)
-		(property "Reference" "#PWR03"
+		(property "Reference" "#PWR024"
 			(at 119.38 86.36 0)
 			(effects
@@
 			(project ""
 				(path "/3902e32d-76e7-44cb-8277-c0e17db8d088/d1d82891-0be9-49d5-808b-34296a85b88c"
-					(reference "#PWR03")
+					(reference "#PWR024")
 					(unit 1)
 				)
@@
 		(dnp no)
 		(fields_autoplaced yes)
-		(property "Reference" "#PWR06"
+		(property "Reference" "#PWR025"
 			(at 139.7 93.98 0)
 			(effects
@@
 			(project "NovaPlay3"
 				(path "/3902e32d-76e7-44cb-8277-c0e17db8d088/d1d82891-0be9-49d5-808b-34296a85b88c"
-					(reference "#PWR06")
+					(reference "#PWR025")
 					(unit 1)
 				)
@@
 		(dnp no)
 		(fields_autoplaced yes)
-		(property "Reference" "#PWR05"
+		(property "Reference" "#PWR027"
 			(at 119.38 115.57 0)
 			(effects
@@
 			(project ""
 				(path "/3902e32d-76e7-44cb-8277-c0e17db8d088/d1d82891-0be9-49d5-808b-34296a85b88c"
-					(reference "#PWR05")
-					(unit 1)
-				)
+					(reference "#PWR027")
+					(unit 1)
+				)
