File: NovaPlay3_KiCad/Power_management.kicad_sch (KiCad schematic)
At the start: 0 parts

Commit message: Finished power management
power management schematic is done
Parts:
- added BT1: Battery_Cell, symbol Device:Battery_Cell
- added C1, C2: 4.7uF, symbol Device:C
- added C3: 10uF, symbol Device:C_Polarized
- added C4: 22uF, symbol Device:C_Polarized
- added C5: 100uF, symbol Device:C_Polarized
- added D1: LED, symbol Device:LED
- added J1: USB_C_Receptacle_USB2.0_14P, symbol Connector:USB_C_Receptacle_USB2.0_14P
- added R1, R3: 33K, symbol Device:R
- added R4: 2K, symbol Device:R
- added R5: 470, symbol Device:R
- added R6: 3k, symbol Device:R
- added R7: 10k, symbol Device:R
- added R8: 100K, symbol Device:R
- added U3: MCP73831-2-MC, Package_DFN_QFN:DFN-8-1EP_3x2mm_P0.5mm_EP1.7x1.4mm, symbol Battery_Management:MCP73831-2-MC
- added U4: MIC5219-3.3YM5, Package_TO_SOT_SMD:SOT-23-5, symbol Regulator_Linear:MIC5219-3.3YM5
Connections:
- new net: D1.1 (K), R5.1
- new net: R8.2, U4.4 (BP)
- new net: R4.1, U3.8 (PROG)
- new net: J1.A5 (CC1), R3.1
- new net: J1.B5 (CC2), R1.1
- new net +3.3V: C4.1, C5.1, U4.5 (OUT)
- new net +5V: C1.1, D1.2 (A), J1.A4 (VBUS), J1.A9 (VBUS), J1.B4 (VBUS), J1.B9 (VBUS), U3.1 (V_{DD}), U3.2 (V_{DD})
- new net +BATT: BT1.1 (+), C2.1, C3.1, R6.1, R8.1, U3.3 (V_{BAT}), U3.4 (V_{BAT}), U4.1 (IN), U4.3 (EN)
- new net BATT_CHRG_STAT: R5.2, U3.5 (STAT)
- new net BATT_LVL_SENSE: R6.2, R7.1
- new net GND: BT1.2 (-), C1.2, C2.2, C3.2, C4.2, C5.2, J1.A1 (GND), J1.A12 (GND), J1.B1 (GND), J1.B12 (GND), J1.S1 (SHIELD), R1.2, R3.2, R4.2, R7.2, U3.6 (V_{SS}), U4.2 (GND)
- new net USB_D+: J1.A6 (D+), J1.B6 (D+)
- new net USB_D-: J1.A7 (D-), J1.B7 (D-)
Other:
- note added: "Battery management"
- note added: "USB-C Power and Data"
- note added: "Voltage divider for battery level sensing"
- note added: "Voltage regulation and smoothing"

Commit message: Sync
Parts:
- added Q1, Q2: MOSFET, symbol Connector_Generic:Conn_02x03_Counter_Clockwise
- added R10, R11: 10K, symbol Device:R
- added R12, R9: 1K, symbol Device:R
- renumbered C5 to C3, C3 to C4, C4 to C5, R1 to R2, R5 to R4, R4 to R5, R8 to R7, R7 to R8, U3 to U2, U4 to U3
Connections:
- net +3.3V: now also Q1.1 (Pin_1), Q1.2 (Pin_2), Q1.5 (Pin_5), Q1.6 (Pin_6)
- net GND: now also Q2.4 (Pin_4), R10.1, R11.1; no longer R8.2
- new net: Q2.1 (Pin_1), Q2.2 (Pin_2), Q2.5 (Pin_5), Q2.6 (Pin_6), R8.2
- new net: Q2.3 (Pin_3), R12.2
- new net: Q1.3 (Pin_3), R9.2
- new net 3.3V_REG: Q1.4 (Pin_4)
- new net MAIN_POWER_EN: R10.2, R11.2, R12.1, R9.1
Other:
- note added: "Main power switching"
- moved on the sheet: R6, R8
